File: bldc_controller/_autosave-bldc_controller.kicad_sch (KiCad schematic)
At the start: 0 parts

Commit message: first commit, schematic not complete yet
Other:
- sheet Motor Control Top Level renamed Motor Control
- sheet Motor Control: file MotorControl_TopLevel.kicad_sch -> MotorControl.kicad_sch
- note added: "11"
- note removed: "11-14"
Changed lines of the file:
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@@
     (effects (font (size 2.54 2.54) bold (color 60 60 120 1)) (justify right bottom) (href "#15"))
   )
-  (text "11-14" (at 219.71 119.38 0)
+  (text "11" (at 219.71 119.38 0)
     (effects (font (size 2.54 2.54) bold (color 100 30 50 1)) (justify right bottom) (href "#11"))
   )
@@
     (stroke (width 0.1524) (type solid))
     (fill (color 255 128 128 0.5000))
-    (property "Sheetname" "Motor Control Top Level" (at 185.42 51.0409 0)
-      (effects (font (size 1.905 1.905) bold) (justify left bottom))
-    )
-    (property "Sheetfile" "MotorControl_TopLevel.kicad_sch" (at 185.42 121.2346 0)
-      (effects (font (size 1.27 1.27)) (justify left top))
-    )
+    (property "Sheetname" "Motor Control" (at 185.42 51.0409 0)
+      (effects (font (size 1.905 1.905) bold) (justify left bottom))
+    )
+    (property "Sheetfile" "MotorControl.kicad_sch" (at 185.42 121.2346 0)
+      (effects (font (size 1.27 1.27)) (justify left top))
+    )
