File: bldc_controller/PositionSensor.kicad_sch (KiCad schematic)
At the start: 3 parts, among them U3 AS5047P

Commit message: some progress
Changed lines of the file:
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@@
     (comment 3 "Author: Vincent Nguyen")
   )
+  (junction (at 130.81 68.58) (diameter 0) (color 0 0 0 0)
+  )
   (junction (at 111.76 110.49) (diameter 0) (color 0 0 0 0)
   )
-  (junction (at 138.43 68.58) (diameter 0) (color 0 0 0 0)
+  (junction (at 140.97 68.58) (diameter 0) (color 0 0 0 0)
   )
   (junction (at 111.76 68.58) (diameter 0) (color 0 0 0 0)
@@
     (stroke (width 0) (type default))
   )
+  (wire (pts (xy 130.81 68.58) (xy 133.35 68.58))
+    (stroke (width 0) (type default))
+  )
   (wire (pts (xy 152.4 86.36) (xy 175.26 86.36))
     (stroke (width 0) (type default))
@@
     (stroke (width 0) (type default))
   )
-  (wire (pts (xy 140.97 77.47) (xy 140.97 81.28))
+  (wire (pts (xy 130.81 77.47) (xy 138.43 77.47))
     (stroke (width 0) (type default))
   )
@@
     (stroke (width 0) (type default))
   )
+  (wire (pts (xy 138.43 68.58) (xy 140.97 68.58))
+    (stroke (width 0) (type default))
+  )
   (wire (pts (xy 111.76 68.58) (xy 111.76 90.17))
     (stroke (width 0) (type default))
@@
     (stroke (width 0) (type default))
   )
-  (wire (pts (xy 138.43 68.58) (xy 138.43 81.28))
+  (wire (pts (xy 130.81 68.58) (xy 130.81 77.47))
     (stroke (width 0) (type default))
   )
@@
     (stroke (width 0) (type default))
   )
-  (wire (pts (xy 138.43 68.58) (xy 140.97 68.58))
-    (stroke (width 0) (type default))
-  )
   (wire (pts (xy 111.76 66.04) (xy 111.76 68.58))
     (stroke (width 0) (type default))
@@
     (stroke (width 0) (type default))
   )
-  (wire (pts (xy 140.97 68.58) (xy 140.97 72.39))
-    (stroke (width 0) (type default))
-  )
-  (wire (pts (xy 111.76 68.58) (xy 138.43 68.58))
-    (stroke (width 0) (type default))
-  )
   (wire (pts (xy 152.4 93.98) (xy 175.26 93.98))
     (stroke (width 0) (type default))
   )
+  (wire (pts (xy 111.76 68.58) (xy 130.81 68.58))
+    (stroke (width 0) (type default))
+  )
+  (wire (pts (xy 138.43 77.47) (xy 138.43 81.28))
+    (stroke (width 0) (type default))
+  )
   (wire (pts (xy 139.7 110.49) (xy 158.75 110.49))
+    (stroke (width 0) (type default))
+  )
+  (wire (pts (xy 140.97 68.58) (xy 140.97 81.28))
     (stroke (width 0) (type default))
   )
@@
     )
   )
-  (symbol (lib_id "Device:R_Small") (at 140.97 74.93 0) (unit 1)
-    (in_bom yes) (on_board yes) (dnp no)
-    (property "Reference" "R21" (at 142.24 73.66 0)
-      (effects (font (size 1.27 1.27)) (justify left))
-    )
-    (property "Value" "0R" (at 142.24 76.2 0)
-      (effects (font (size 1.27 1.27)) (justify left))
-    )
-    (property "Footprint" "" (at 140.97 74.93 0)
-      (effects (font (size 1.27 1.27)) hide)
-    )
-    (property "Datasheet" "~" (at 140.97 74.93 0)
+  (symbol (lib_id "Device:R_Small") (at 135.89 68.58 90) (unit 1)
+    (in_bom yes) (on_board yes) (dnp no) (fields_autoplaced)
+    (property "Reference" "R21" (at 135.89 63.5 90)
+      (effects (font (size 1.27 1.27)))
+    )
+    (property "Value" "0R" (at 135.89 66.04 90)
+      (effects (font (size 1.27 1.27)))
+    )
+    (property "Footprint" "" (at 135.89 68.58 0)
+      (effects (font (size 1.27 1.27)) hide)
+    )
+    (property "Datasheet" "~" (at 135.89 68.58 0)
       (effects (font (size 1.27 1.27)) hide)
     )
@@
         )
       )
+    )
+  )
+  (symbol (lib_id "power:PWR_FLAG") (at 140.97 68.58 0) (unit 1)
+    (in_bom yes) (on_board yes) (dnp no) (fields_autoplaced)
+    (property "Reference" "#FLG05" (at 140.97 66.675 0)
+      (effects (font (size 1.27 1.27)) hide)
+    )
+    (property "Value" "PWR_FLAG" (at 140.97 63.5 0)
+      (effects (font (size 1.27 1.27)) hide)
+    )
+    (property "Footprint" "" (at 140.97 68.58 0)
+      (effects (font (size 1.27 1.27)) hide)
+    )
+    (property "Datasheet" "~" (at 140.97 68.58 0)
+      (effects (font (size 1.27 1.27)) hide)
+    )
+    (pin "1")
+    (instances
+      (project "bldc_controller"
+        (path "/0650c7a8-acba-429c-9f8e-eec0baf0bc1c/aba936fa-d9e9-4532-8179-f8f593419a0b"
+          (reference "#FLG05") (unit 1)
+        )
+      )
