File: bldc_controller/Interconnects.kicad_sch (KiCad schematic)
At the start: 53 parts, among them J10 JST S2B-PH-SM4-TB, J3 SM08B-GHS-TB, J4 SM07B-GHS-TB, J5 JST S2B-PH-SM4-TB, J6 SM06B-GHS-TB, J7 Nano-Fit 1x03, J8 Nano-Fit 1x03, J9 SM05B-GHS-TB, SW1 CAS-220TA

Commit message: might have fixed net issue, added dxf and svgs
Parts:
- removed J4: SM07B-GHS-TB, Connector_JST:JST_GH_SM07B-GHS-TB_1x07-1MP_P1.25mm_Horizontal, symbol Connector_Generic:Conn_01x07
- removed J9: SM05B-GHS-TB, Connector_JST:JST_GH_SM05B-GHS-TB_1x05-1MP_P1.25mm_Horizontal, symbol Connector_Generic:Conn_01x05
- added J4: SM07B-GHS-TB, Connector_JST:JST_GH_SM07B-GHS-TB_1x07-1MP_P1.25mm_Horizontal, symbol 0_connectors:Conn_01x07_Shield
- added J9: SM05B-GHS-TB, Connector_JST:JST_GH_SM05B-GHS-TB_1x05-1MP_P1.25mm_Horizontal, symbol 0_connectors:Conn_01x05_Shield
- R23, R24: value 120R -> 100R
- gave numbers to parts that had none: 4
Connections:
- net +3V3: now also J4.2 (Pin_2), J9.1 (Pin_1)
- net +5V: now also J4.1 (Pin_1)
- net AUX2P_A: now also J4.3 (Pin_3)
- net AUX2P_B: now also J4.4 (Pin_4)
- net AUX2P_C: now also J4.5 (Pin_5)
- net AUX2P_D: now also J4.6 (Pin_6)
- net GND: now also J4.7 (Pin_7), J9.5 (Pin_5)
- net NRST: now also J9.4 (Pin_4)
- net SWCLK: now also J9.3 (Pin_3)
- net SWDIO: now also J9.2 (Pin_2)
- new net CHASSIS: J4.MP, J9.MP
Other:
- moved on the sheet: C73, C74, C75, C76, C77, C78, C79, C80, C81, C82, C83, C84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
