File: bldc_controller/Interface - Interconnects.kicad_sch (KiCad schematic)
At the start: 54 parts, among them J10 JST S2B-PH-SM4-TB, J11 Nano-Fit 1x03, J12 Nano-Fit 1x03, J13 SM05B-GHS-TB, J14 PTH 01x02 2.54mm, J6 SM08B-GHS-TB, J7 SM07B-GHS-TB, J8 JST S2B-PH-SM4-TB, J9 SM06B-GHS-TB, SW1 CAS-220TA

Commit message: schematic is complete. Replaced 5V buck and added pi filters.
Parts:
- added C123, C98, C99: 100n X7R 100V, 0_capacitor_smd:C_0402_1005_DensityHigh, symbol Device:C_Small
- C105, C106, C107, C108, C118: value 100n -> 100n X7R 100V
- C119: value 4u7 -> 4u7 X7R 25V
Connections:
- net +12V: now also C123.1
- net +3V3: now also C99.1
- net +5V: now also C98.1
- net GND: now also C123.2, C98.2, C99.2
Other:
- moved on the sheet: C105, C106, C107, C108, C109, C110, C111, C112, C113, C114, C115, C116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

Commit message: added assembly files
Parts:
- R30, R31, R32, R33, R34, R35, R36, R37, R38, R45, R46: value 100R -> 100R 1%
- R39, R40, R41, R42: value 2k -> 2k 1%
- R43, R44: value 60R -> 60R4 1% 1/4W
Other:
- moved on the sheet: C119, R45, R46
