File: amulet_controller/Power - Generation.kicad_sch (KiCad schematic)
At the start: 90 parts, among them U2 LMR36503MSC5RPERQ1, U3 LMR36006FSCQRNXRQ1, U4 TPS62172DSG, U5 LP2992IM5-3.3/NOPB

Commit message: filled in fields for bom, replaced inexisting components. Need to replace LEDs
Parts:
- removed U3: LMR36006FSCQRNXRQ1, 0_switching_regulator:LMR36006FSCQRNXRQ1, symbol 0_switching_regulator:LMR36006FSCQRNXRQ1
- added U3: LMR36006FSCQ, 0_switching_regulator:LMR36006, symbol 0_switching_regulator:LMR36006FSCQ
- C124, C125, C126, C127, C128, C129, C17: Manufacturer (none) -> TDK Corporation; Manufacturer Part Number (none) -> CGA4J1X7R2A225K125AC; Supplier 1 (none) -> Mouser; Supplier Part Number 1 (none) -> 810-CGA4J7R2A225K125
- C131, C54, C58: value 100n X7R 100V -> 100n X7R 50V; Manufacturer (none) -> Murata Electronics; Manufacturer Part Number (none) -> GCM155R71H104KE02J; Supplier 1 (none) -> Digikey; Supplier Part Number 1 (none) -> 490-14514-1-ND
- C132: footprint 0_capacitor_smd:C_0402_1005_DensityHigh -> 0_capacitor_smd:C_0603_1608_DensityHigh; Manufacturer (none) -> Taiyo Yuden; Manufacturer Part Number (none) -> HMK107B7104KAHT; Supplier 1 (none) -> Digikey; Supplier Part Number 1 (none) -> 587-6009-1-ND
- C14, C15, C16, C18, C19, C20, C21, C22, C23, C24, C25, C26, C27, C28, C30, C31, C32, C34, C35, C36, C38, C39, C40, C42, C43, C44, C45, C46, C47, C48, C49, C50, C51, C52, C53, C55, C56, C57, C59, C60, C61, C63, C64, C65, C66, C67, C68, C70, C71, C72: Manufacturer (none) -> Murata Electronics; Manufacturer Part Number (none) -> GRJ31CZ72A475KE01L; Supplier 1 (none) -> Digikey; Supplier Part Number 1 (none) -> 490-GRJ31CZ72A475KE01LCT-ND
- C29, C37: value 220n X7R 100V -> 220n X7S 100V; footprint 0_capacitor_smd:C_0402_1005_DensityHigh -> 0_capacitor_smd:C_0603_1608_DensityHigh; Manufacturer (none) -> Taiyo Yuden; Manufacturer Part Number (none) -> HMK107C7224KAHTE; Supplier 1 (none) -> Digikey; Supplier Part Number 1 (none) -> 587-5012-1-ND
- C33, C41: value 1u X7R 100V -> 1u X7R 10V; Manufacturer (none) -> Murata Electronics; Manufacturer Part Number (none) -> GRM155Z71A105KE01J; Supplier 1 (none) -> Digikey; Supplier Part Number 1 (none) -> 490-GRM155Z71A105KE01JCT-ND
- C62: value 10u X7R 6.3V -> 10u X7R 25V; Manufacturer (none) -> Murata Electronics; Manufacturer Part Number (none) -> GRM21BZ71E106KE15L; Supplier 1 (none) -> Digikey; Supplier Part Number 1 (none) -> 490-GRM21BZ71E106KE15LCT-ND
- C69, C73: Manufacturer (none) -> TDK Corporation; Manufacturer Part Number (none) -> CGA6M3X7R1E156M200AB; Supplier 1 (none) -> Digikey; Supplier Part Number 1 (none) -> 445-175431-1-ND
- C74: value 10u X7R 6.3V -> 1u X7R 25V; footprint 0_capacitor_smd:C_0805_2012_DensityHighest -> 0_capacitor_smd:C_0603_1608_DensityHigh; Manufacturer (none) -> Taiyo Yuden; Manufacturer Part Number (none) -> TMK107AB7105KAHT; Supplier 1 (none) -> Digikey; Supplier Part Number 1 (none) -> 587-3467-1-ND
- C75: Manufacturer (none) -> Murata Electronics; Manufacturer Part Number (none) -> GRM21BZ71E106KE15L; Supplier 1 (none) -> Digikey; Supplier Part Number 1 (none) -> 490-GRM21BZ71E106KE15LCT-ND
- C76: value 10n X7R 25V -> 10n X7R 100V; Manufacturer (none) -> Taiyo Yuden; Manufacturer Part Number (none) -> HMR105B7103KV-F; Supplier 1 (none) -> Digikey; Supplier Part Number 1 (none) -> 587-HMR105B7103KV-FCT-ND
- C77: value 10u X7R 6.3V -> 4u7 X7R 16V; footprint 0_capacitor_smd:C_0805_2012_DensityHighest -> 0_capacitor_smd:C_0603_1608_DensityHigh; Manufacturer (none) -> Murata Electronics; Manufacturer Part Number (none) -> GRM188Z71C475KE21J; Supplier 1 (none) -> Digikey; Supplier Part Number 1 (none) -> 490-GRM188Z71C475KE21JCT-ND
- C78: Manufacturer (none) -> Murata Electronics; Manufacturer Part Number (none) -> GRM21BZ71A226ME15L; Supplier 1 (none) -> Digikey; Supplier Part Number 1 (none) -> 490-GRM21BZ71A226ME15LCT-ND
- FB1, FB2, FB3: Manufacturer (none) -> Würth Elektronik; Supplier 1 (none) -> Digikey; Supplier Part Number 1 (none) -> 732-4648-1-ND
- L1, L2: Manufacturer (none) -> Coilcraft
- L3: Manufacturer (none) -> Coilcraft; Supplier 1 (none) -> Mouser; Supplier Part Number 1 (none) -> 994-LPS3314-222MRC
- R28: Manufacturer (none) -> YAGEO; Manufacturer Part Number (none) -> RT0402FRE0710KL; Supplier 1 (none) -> Digikey; Supplier Part Number 1 (none) -> YAG1233CT-ND
- R4: Manufacturer (none) -> Panasonic Electronic Components; Manufacturer Part Number (none) -> ERJ-2GE0R00X; Supplier 1 (none) -> Digikey; Supplier Part Number 1 (none) -> P0.0JCT-ND
- R5: Manufacturer (none) -> YAGEO; Manufacturer Part Number (none) -> RT0402FRE07100KL; Supplier 1 (none) -> Digikey; Supplier Part Number 1 (none) -> YAG2307CT-ND
- R6: Manufacturer (none) -> YAGEO; Manufacturer Part Number (none) -> RT0402FRE079K09L; Supplier 1 (none) -> Digikey; Supplier Part Number 1 (none) -> 13-RT0402FRE079K09LCT-ND
- U2: Height 0.9 -> (none); Manufacturer (none) -> Texas Instruments; Manufacturer Part Number (none) -> LMR36503MSC5RPERQ1; Manufacturer_Name Texas Instruments -> (none); Manufacturer_Part_Number LMR36006FSCQRNXRQ1 -> (none); Mouser Part Number 595-R36006FSCQRNXRQ1 -> (none); Mouser Price/Stock https://www.mouser.co.uk/ProductDetail/Texas-Instruments/LM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 -> (none); Supplier 1 (none) -> Digikey; Supplier Part Number 1 (none) -> 296-LMR36503MSC5RPERQ1CT-ND
- U4: Manufacturer (none) -> Texas Instruments; Manufacturer Part Number (none) -> TPS62172DSGR; Supplier 1 (none) -> Digikey; Supplier Part Number 1 (none) -> 296-39449-1-ND
- U5: Manufacturer (none) -> Texas Instruments; Manufacturer Part Number (none) -> LP2992IM5-3.3/NOPB; Supplier 1 (none) -> Digikey; Supplier Part Number 1 (none) -> LP2992IM5-3.3/NOPBCT-ND
Connections:
- net BOOT_12V: now also U3.4 (BOOT)
- net FB_DIV_12V: now also U3.7 (FB)
- net F_VIN_12V: now also U3.10 (VIN), U3.2 (VIN), U3.9 (EN)
- net GND: now also U3.1 (PGND), U3.11 (PGND), U3.6 (AGND)
- net PG_12V: now also U3.8 (PG)
- net SW_12V: now also U3.12 (SW), U3.3 (NC)
- net VCC_12V: now also U3.5 (VCC)
Other:
- moved on the sheet: C124, C125, C74, C75, C76, C77, C78, FB3, L3, NT3, U4, U5

Commit message: added test points
Parts:
- added TP1 (x3): +VBAT, 0_testpoint:TestPoint_Pad_D0.5mm_Front, symbol Connector:TestPoint
- added TP1 (x5): GND, 0_testpoint:TestPoint_Pad_D0.5mm_Front, symbol Connector:TestPoint
- added TP1: +5V, 0_testpoint:TestPoint_Pad_D0.5mm_Front, symbol Connector:TestPoint
- added TP1: +A3V3, 0_testpoint:TestPoint_Pad_D0.5mm_Front, symbol Connector:TestPoint
- added TP1: F_VIN_5V, 0_testpoint:TestPoint_Pad_D0.5mm_Front, symbol Connector:TestPoint
- added TP1: F_VIN_3V3, 0_testpoint:TestPoint_Pad_D0.5mm_Back, symbol Connector:TestPoint
- added TP1: +12V, 0_testpoint:TestPoint_Pad_D0.5mm_Front, symbol Connector:TestPoint
- added TP1: +3V3, 0_testpoint:TestPoint_Pad_D0.5mm_Front, symbol Connector:TestPoint
- added TP1: F_VIN_12V, 0_testpoint:TestPoint_Pad_D0.5mm_Front, symbol Connector:TestPoint
Connections:
- net +12V: now also TP1.1
- net +3V3: now also TP1.1
- net +5V: now also TP1.1
- net +A3V3: now also TP1.1
- net +VBAT: now also TP1.1, TP1.1, TP1.1
- net F_VIN_12V: now also TP1.1
- net F_VIN_3V3: now also TP1.1
- net F_VIN_5V: now also TP1.1
- net GND: now also TP1.1, TP1.1, TP1.1, TP1.1, TP1.1

Commit message: finalized pcb. TODO: add clean BOM and KiBot integration
Parts:
- added TP1: GND, 0_testpoint:TestPoint_Pad_D0.5mm_Back, symbol Connector:TestPoint
- added TP1: GND, 0_testpoint:TestPoint_Pad_D0.5mm_Front, symbol Connector:TestPoint
- added TP1: +5V, 0_testpoint:TestPoint_Pad_D0.5mm_Back, symbol Connector:TestPoint
- added TP1: +3V3, 0_testpoint:TestPoint_Pad_D0.5mm_Front, symbol Connector:TestPoint
- added TP1: +3V3, 0_testpoint:TestPoint_Pad_D0.5mm_Back, symbol Connector:TestPoint
- renumbered C128 to C15, C127 to C16, C129 to C17, C126 to C18, C18 to C19, C17 to C20, C25 to C21, C132 to C22, C29 to C23, C33 to C24, C37 to C25, C41 to C26, C131 to C27, C58 to C28, C54 to C29, C69 to C30, C14 to C31, C15 to C32, C16 to C33, C19 to C34, C20 to C35, C21 to C36, C62 to C37, C73 to C38, C22 to C39, C23 to C40, C24 to C41, C26 to C42, C27 to C43, C28 to C44, C125 to C45, C30 to C46, C31 to C47, C32 to C48, C34 to C49, C35 to C50, C36 to C51, C124 to C52, C38 to C53, C39 to C54, C40 to C55, C75 to C56, C42 to C57, C43 to C58, C44 to C59, C74 to C60, C45 to C61, C46 to C62, C47 to C63, C48 to C64, C49 to C65, C50 to C66, C51 to C67, C52 to C68, C53 to C69, C55 to C70, C56 to C71, C57 to C72, C59 to C73, C60 to C74, C61 to C75, C63 to C77, C64 to C78, C65 to C79, C66 to C80, C67 to C81, C68 to C82, C78 to C83, C77 to C84, C70 to C85, C71 to C86, C72 to C87, FB1 to FB3, FB3 to FB4
Connections:
- net +3V3: now also TP1.1, TP1.1
- net +5V: now also TP1.1
- net GND: now also TP1.1, TP1.1
Other:
- moved on the sheet: TP1
