File: amulet_controller/Project Architecture.kicad_sch (KiCad schematic)
At the start: 0 parts

Commit message: small typos
Other:
- sheet Misc - Board Version Divider, DAC renamed Misc - Board Version, DAC
- sheet Misc - Board Version, DAC: file Misc - Board Version Divider DAC.kicad_sch -> Misc - Board Version DAC.kicad_sch
Changed lines of the file:
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@@
     (stroke (width 0.1524) (type solid))
     (fill (color 255 255 150 0.5000))
-    (property "Sheetname" "Misc - Board Version Divider, DAC" (at 248.92 171.6909 0)
+    (property "Sheetname" "Misc - Board Version, DAC" (at 248.92 171.6909 0)
       (effects (font (size 1.905 1.905) bold) (justify left bottom))
     )
-    (property "Sheetfile" "Misc - Board Version Divider DAC.kicad_sch" (at 248.92 183.4646 0)
+    (property "Sheetfile" "Misc - Board Version DAC.kicad_sch" (at 248.92 183.4646 0)
       (effects (font (face "Arial") (size 1.27 1.27)) (justify left top))
     )

Commit message: updated documents
Other:
- sheet Mechanical - Holes renamed Misc - Holes, Fiducials
- sheet Misc - Holes, Fiducials: file Mechanical - Holes.kicad_sch -> Misc - Holes Fiducials.kicad_sch
Changed lines of the file:
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@@
   (title_block
     (title "Project Architecture")
-    (date "2023-11-25")
+    (date "2023-12-22")
     (rev "${REVISION}")
     (company "${COMPANY}")
@@
     (stroke (width 0) (type default))
   )
-  (polyline (pts (xy 124.46 92.71) (xy 124.46 76.2))
+  (polyline (pts (xy 124.46 104.14) (xy 124.46 76.2))
     (stroke (width 0) (type default))
   )
@@
     (stroke (width 0) (type default))
   )
-  (polyline (pts (xy 124.46 179.705) (xy 124.46 236.22))
+  (polyline (pts (xy 124.46 191.008) (xy 124.46 236.22))
     (stroke (width 0) (type default))
   )
@@
     (stroke (width 0) (type default))
   )
-  (polyline (pts (xy 124.46 120.65) (xy 124.46 177.165))
+  (polyline (pts (xy 124.46 144.145) (xy 124.46 188.468))
     (stroke (width 0) (type default))
   )
@@
     (stroke (width 0) (type default))
   )
-  (polyline (pts (xy 124.46 95.25) (xy 124.46 111.76))
+  (polyline (pts (xy 124.46 106.68) (xy 124.46 135.89))
     (stroke (width 0) (type default))
   )
@@
     (fill (type none))
   )
-  (arc (start 124.46 92.71) (mid 124.0851 93.6051) (end 123.19 93.98)
+  (arc (start 124.46 104.14) (mid 124.0851 105.0351) (end 123.19 105.41)
     (stroke (width 0) (type default))
     (fill (type none))
@@
     (fill (type none))
   )
-  (arc (start 124.46 177.165) (mid 124.0834 178.0569) (end 123.19 178.435)
+  (arc (start 124.46 188.468) (mid 124.084 189.3634) (end 123.19 189.738)
     (stroke (width 0) (type default))
     (fill (type none))
@@
     (fill (type none))
   )
-  (arc (start 124.46 120.65) (mid 125.2039 118.8539) (end 127 118.11)
+  (arc (start 124.46 144.145) (mid 125.2039 142.3489) (end 127 141.605)
     (stroke (width 0) (type default))
     (fill (type none))
@@
     (fill (type none))
   )
-  (arc (start 123.19 93.98) (mid 124.0851 94.3549) (end 124.46 95.25)
+  (arc (start 123.19 105.41) (mid 124.0851 105.7849) (end 124.46 106.68)
     (stroke (width 0) (type default))
     (fill (type none))
@@
     (fill (type none))
   )
-  (arc (start 123.19 178.435) (mid 124.0869 178.8096) (end 124.46 179.705)
+  (arc (start 123.19 189.738) (mid 124.0834 190.1132) (end 124.46 191.008)
     (stroke (width 0) (type default))
     (fill (type none))
@@
     (fill (type none))
   )
-  (arc (start 127 114.3) (mid 125.2098 113.5502) (end 124.46 111.76)
+  (arc (start 127 138.43) (mid 125.2098 137.6802) (end 124.46 135.89)
     (stroke (width 0) (type default))
     (fill (type none))
@@
     (effects (font (size 1.905 1.905) (thickness 0.381) bold (color 0 0 0 1)) (justify right top))
   )
-  (text_box "Peripherals\nSensors"
-    (at 102.87 173.355 0) (size 19.685 10.16)
+  (text_box "Interfaces"
+    (at 102.87 186.69 0) (size 19.685 10.16)
     (stroke (width -0.0001) (type default))
     (fill (type none))
@@
   )
   (text_box "Sensing"
-    (at 109.22 91.44 0) (size 13.335 5.08)
+    (at 109.22 102.87 0) (size 13.335 5.08)
     (stroke (width -0.0001) (type default))
     (fill (type none))
@@
     (effects (font (face "Times New Roman") (size 8 8) (thickness 1.2) bold (color 162 22 34 1)))
   )
-  (text_box "LEDs, version"
-    (at 299.085 164.465 0) (size 13.335 7.62)
+  (text_box "LEDs\nBoard version"
+    (at 299.085 164.465 0) (size 20.955 7.62)
     (stroke (width -0.0001) (type default))
     (fill (type none))
     (effects (font (size 1.905 1.905) (thickness 0.381) bold (color 0 0 0 1)) (justify left top))
   )
-  (text_box "Mounting holes\nTest pads"
+  (text_box "Mounting holes\nFiducial markers"
     (at 298.45 222.25 0) (size 26.015 10.18)
     (stroke (width -0.0001) (type default))
@@
     (effects (font (size 1.905 1.905) (thickness 0.381) bold (color 0 0 0 1)) (justify left top))
   )
-  (text_box "Gate driver\n3-Phase inverter"
+  (text_box "Gate driver\n3-phase inverter"
     (at 298.45 105.41 0) (size 29.21 10.16)
     (stroke (width -0.0001) (type default))
@@
     (stroke (width 0.1524) (type solid))
     (fill (color 0 0 0 0.1200))
-    (property "Sheetname" "Mechanical - Holes" (at 248.92 216.1409 0)
-      (effects (font (size 1.905 1.905) bold) (justify left bottom))
-    )
-    (property "Sheetfile" "Mechanical - Holes.kicad_sch" (at 248.92 238.0746 0)
-      (effects (font (face "Arial") (size 1.27 1.27)) (justify left top))
-    )
+    (property "Sheetname" "Misc - Holes, Fiducials" (at 248.92 216.1409 0)
+      (effects (font (size 1.905 1.905) bold) (justify left bottom))
+    )
+    (property "Sheetfile" "Misc - Holes Fiducials.kicad_sch" (at 248.92 238.0746 0)
+      (effects (font (face "Arial") (size 1.27 1.27)) (justify left top))
+    )
