File: smps_legged_robot/SMPS_Motherboard/Block Diagram.kicad_sch (KiCad schematic)
At the start: 0 parts

Commit message: Buck module finished pending review
Other:
- note added: "+12V"
- note added: "+3V3"
- note added: "+5V"
- note added: "+VBAT"
- note removed: "+??V"
- note removed: "+A3V3"
