File: smps_legged_robot/SMPS_Motherboard/smps_legged_robot.kicad_pcb (KiCad board)
At the start: 6 copper layers, 0 parts

Commit message: Buck module finished pending review
Parts:
- added C1101: 100n X7R 50V, 0_capacitor_smd:C_0402_1005_DensityHigh, F.Cu at (129.1, 43.7)
- added C1102: 100n X7R 50V, 0_capacitor_smd:C_0402_1005_DensityHigh, F.Cu at (177.4, 48.4)
- added C1103: 100n X7R 50V, 0_capacitor_smd:C_0402_1005_DensityHigh, B.Cu at (91.1, 60.0)
- added C1104: 100n X7R 50V, 0_capacitor_smd:C_0402_1005_DensityHigh, F.Cu at (132.7, 45.9)
- added C1105: 100n X7R 50V, 0_capacitor_smd:C_0402_1005_DensityHigh, F.Cu at (170.3, 83.9)
- added C1106: 100n X7R 50V, 0_capacitor_smd:C_0402_1005_DensityHigh, B.Cu at (89.8, 60.0)
- added C1107: 100n X7R 50V, 0_capacitor_smd:C_0402_1005_DensityHigh, B.Cu at (65.0, 60.0)
- added C1108: 100n X7R 50V, 0_capacitor_smd:C_0402_1005_DensityHigh, B.Cu at (63.8, 60.0)
- added C1109: 100n X7R 50V, 0_capacitor_smd:C_0402_1005_DensityHigh, F.Cu at (157.4, 88.7)
- added C1110: 100n X7R 50V, 0_capacitor_smd:C_0402_1005_DensityHigh, F.Cu at (144.1, 89.8)
- added C1111: 1u X7R 50V, 0_capacitor_smd:C_0402_1005_DensityHigh, F.Cu at (144.1, 91.7)
- added C1112: 100n X7R 50V, 0_capacitor_smd:C_0402_1005_DensityHigh, F.Cu at (149.0, 84.5)
- added C1113: 100n X7R 50V, 0_capacitor_smd:C_0402_1005_DensityHigh, F.Cu at (144.1, 93.6)
- added C1114: 220p X7R 50V, 0_capacitor_smd:C_0402_1005_DensityHigh, F.Cu at (144.1, 90.7)
- added C1115: 100n X7R 50V, 0_capacitor_smd:C_0402_1005_DensityHigh, F.Cu at (151.6, 84.5)
- added C1116: 100n X7R 50V, 0_capacitor_smd:C_0402_1005_DensityHigh, F.Cu at (144.1, 94.7)
- added C1117: 100n X7R 50V, 0_capacitor_smd:C_0402_1005_DensityHigh, F.Cu at (150.3, 83.1)
- added C1118: 100n X7R 50V, 0_capacitor_smd:C_0402_1005_DensityHigh, F.Cu at (156.5, 86.4)
- added C1119: 100n X7R 50V, 0_capacitor_smd:C_0402_1005_DensityHigh, F.Cu at (144.1, 86.4)
- added C1120: 100n X7R 50V, 0_capacitor_smd:C_0402_1005_DensityHigh, F.Cu at (157.4, 92.8)
- added C1121: 100n X7R 50V, 0_capacitor_smd:C_0402_1005_DensityHigh, F.Cu at (157.4, 93.7)
- added C1122: 100n X7R 50V, 0_capacitor_smd:C_0402_1005_DensityHigh, F.Cu at (151.5, 98.6)
- added C1123: 100n X7R 50V, 0_capacitor_smd:C_0402_1005_DensityHigh, F.Cu at (154.6, 98.6)
- added C1124: 100n X7R 50V, 0_capacitor_smd:C_0402_1005_DensityHigh, F.Cu at (150.6, 98.6)
- added C1125: 100n X7R 50V, 0_capacitor_smd:C_0402_1005_DensityHigh, F.Cu at (149.9, 84.5)
- added C1126: 100n X7R 50V, 0_capacitor_smd:C_0402_1005_DensityHigh, F.Cu at (154.8, 86.4)
- added C1127: 100n X7R 50V, 0_capacitor_smd:C_0402_1005_DensityHigh, F.Cu at (145.8, 86.4)
- added C1128: 100n X7R 50V, 0_capacitor_smd:C_0402_1005_DensityHigh, F.Cu at (148.6, 98.6)
- added C1129: 15p X7R 50V, 0_capacitor_smd:C_0603_1608_DensityHigh, F.Cu at (157.4, 83.7)
- added C1130: 15p X7R 50V, 0_capacitor_smd:C_0603_1608_DensityHigh, F.Cu at (135.3, 85.9)
- added C1131: 15p X7R 50V, 0_capacitor_smd:C_0603_1608_DensityHigh, F.Cu at (160.0, 83.7)
- added C1132: 15p X7R 50V, 0_capacitor_smd:C_0603_1608_DensityHigh, F.Cu at (137.9, 85.9)
- added C1133: 18p NP0 50V, 0_capacitor_smd:C_0402_1005_DensityHigh, F.Cu at (144.1, 88.9)
- added C1134: 15p X7R 50V, 0_capacitor_smd:C_0603_1608_DensityHigh, F.Cu at (160.5, 86.0)
- added C1135: 15p X7R 50V, 0_capacitor_smd:C_0603_1608_DensityHigh, F.Cu at (138.4, 83.6)
- added C1136: 18p NP0 50V, 0_capacitor_smd:C_0402_1005_DensityHigh, F.Cu at (144.1, 87.3)
- added C1137: 15p X7R 50V, 0_capacitor_smd:C_0603_1608_DensityHigh, F.Cu at (163.1, 86.0)
- added C1138: 15p X7R 50V, 0_capacitor_smd:C_0603_1608_DensityHigh, F.Cu at (141.0, 83.6)
- added C1139: 100n X7R 50V, 0_capacitor_smd:C_0402_1005_DensityHigh, F.Cu at (135.0, 82.9)
- added C1140: 100n X7R 50V, 0_capacitor_smd:C_0402_1005_DensityHigh, F.Cu at (163.5, 83.0)
- added C1141: 22n X7R 50V, 0_capacitor_smd:C_0603_1608_DensityHigh, F.Cu at (165.6, 86.0)
- added C1142: 22n X7R 50V, 0_capacitor_smd:C_0603_1608_DensityHigh, F.Cu at (132.9, 85.9)
- added C1143: 22n X7R 50V, 0_capacitor_smd:C_0603_1608_DensityHigh, F.Cu at (165.6, 84.7)
- added C1144: 22n X7R 50V, 0_capacitor_smd:C_0603_1608_DensityHigh, F.Cu at (132.8, 84.6)
- added C1145: 100n X7R 50V, 0_capacitor_smd:C_0402_1005_DensityHigh, F.Cu at (135.0, 83.9)
- added C1146: 100n X7R 50V, 0_capacitor_smd:C_0402_1005_DensityHigh, F.Cu at (163.5, 84.0)
- added C1147: 100n X7R 50V, 0_capacitor_smd:C_0402_1005_DensityHigh, F.Cu at (161.5, 96.2)
- added C1148: 2.2u X7R 25V, 0_capacitor_smd:C_0805_2012_DensityHigh, F.Cu at (160.1, 96.5)
- added C1149: 4n7 X7R 100V, 0_capacitor_smd:C_0402_1005_DensityHigh, F.Cu at (181.0, 38.4)
- added C1150: 4n7 X7R 100V, 0_capacitor_smd:C_0402_1005_DensityHigh, F.Cu at (125.5, 38.1)
- added C1151: DNP, 0_capacitor_smd:C_0402_1005_DensityHigh, B.Cu at (65.2, 62.2)
- added C1152: DNP, 0_capacitor_smd:C_0402_1005_DensityHigh, B.Cu at (67.7, 62.2)
- added C1153: DNP, 0_capacitor_smd:C_0402_1005_DensityHigh, B.Cu at (68.5, 62.2)
- added C1154: DNP, 0_capacitor_smd:C_0402_1005_DensityHigh, B.Cu at (71.0, 62.2)
- added C1155: DNP, 0_capacitor_smd:C_0402_1005_DensityHigh, B.Cu at (91.3, 62.1)
- added C1156: DNP, 0_capacitor_smd:C_0402_1005_DensityHigh, B.Cu at (93.8, 62.1)
- added C1157: DNP, 0_capacitor_smd:C_0402_1005_DensityHigh, B.Cu at (94.7, 62.1)
- added C1158: DNP, 0_capacitor_smd:C_0402_1005_DensityHigh, B.Cu at (97.1, 62.1)
- added C1201: 2u2 X7R 100V, 0_capacitor_smd:C_0805_2012_DensityHigh, F.Cu at (166.7, 129.8)
- added C1202: 2u2 X7R 100V, 0_capacitor_smd:C_0805_2012_DensityHigh, F.Cu at (166.7, 132.5)
- added C1203: 2u2 X7R 100V, 0_capacitor_smd:C_0805_2012_DensityHigh, F.Cu at (139.0, 145.7)
- added C1204: 100n X7R 100V, 0_capacitor_smd:C_0805_2012_DensityHigh, F.Cu at (137.2, 145.7)
- added C1205: 2.2u X7R 25V, 0_capacitor_smd:C_0805_2012_DensityHigh, F.Cu at (129.1, 150.0)
- added C1206: 100n X7R 50V, 0_capacitor_smd:C_0402_1005_DensityHigh, F.Cu at (129.2, 148.2)
- added C1207: 10u X7R 25V, 0_capacitor_smd:C_1210_3225_DensityHigh, F.Cu at (128.6, 141.4)
- added C1208: 4.7uF X7R 25V, 0_capacitor_smd:C_1210_3225_DensityHigh, F.Cu at (128.0, 137.4)
- added C1209: 1u X7R 25V, 0_capacitor_smd:C_0603_1608_DensityHigh, F.Cu at (134.7, 136.9)
- added C1210: 22u X7R 10V, 0_capacitor_smd:C_1210_3225_DensityHigh, F.Cu at (134.4, 131.5)
- added C1211: 22u X7R 10V, 0_capacitor_smd:C_0805_2012_DensityHigh, F.Cu at (132.2, 134.8)
- added C1301: 100n X7R 50V, 0_capacitor_smd:C_0402_1005_DensityHigh, F.Cu at (188.3, 93.4)
- added C1302: 100n X7R 100V, 0_capacitor_smd:C_0603_1608_DensityHigh, F.Cu at (189.7, 104.2)
- added C1303: 100n X7R 50V, 0_capacitor_smd:C_0402_1005_DensityHigh, F.Cu at (178.5, 93.4)
- added C1305: 100n X7R 50V, 0_capacitor_smd:C_0402_1005_DensityHigh, F.Cu at (188.3, 95.0)
- added C1401: 100n X7R 100V, 0_capacitor_smd:C_0603_1608_DensityHigh, F.Cu at (114.8, 86.6)
- added C1501: 10uF X7R 100V, 0_capacitor_smd:C_1210_3225_DensityHigh, F.Cu at (102.0, 81.1)
- added C1502: 2nF X7R 50V, 0_capacitor_smd:C_1206_3216_DensityHigh, F.Cu at (14.8, 44.5)
- added C1503: 110n X7R 100V, 0_capacitor_smd:C_0603_1608_DensityHigh, F.Cu at (-37.8, 93.5)
- added C1701: 100n X7R 50V, 0_capacitor_smd:C_0402_1005_DensityHigh, F.Cu at (117.9, -17.2)
- added C1702: 4.7n X7R 50V, 0_capacitor_smd:C_0603_1608_DensityHigh, F.Cu at (211.1, -18.0)
- added C1703: 4.7n X7R 50V, 0_capacitor_smd:C_0603_1608_DensityHigh, F.Cu at (211.1, -15.6)
- added C1704: 4.7n X7R 50V, 0_capacitor_smd:C_0603_1608_DensityHigh, F.Cu at (211.1, -13.1)
- added C1705: 470n X5R 16V, 0_capacitor_smd:C_0603_1608_DensityHigh, F.Cu at (203.8, -8.28)
- added C1706: 470n X5R 16V, 0_capacitor_smd:C_0603_1608_DensityHigh, F.Cu at (211.1, -10.6)
- added C1707: 220n X7R 10V, 0_capacitor_smd:C_0603_1608_DensityHigh, F.Cu at (105.3, -19.9)
- added C1708: 1u X7R 16V, 0_capacitor_smd:C_0603_1608_DensityHigh, F.Cu at (105.3, -17.7)
- added C1709: 100n X7R 50V, 0_capacitor_smd:C_0402_1005_DensityHigh, F.Cu at (122.1, -18.0)
- added C1801: 100n X7R 50V, 0_capacitor_smd:C_0402_1005_DensityHigh, F.Cu at (174.8, -8.26)
- added C1802: 4.7u X7R 16V, 0_capacitor_smd:C_0603_1608_DensityHigh, F.Cu at (160.4, -10.5)
- added C2001: 100n X7R 50V, 0_capacitor_smd:C_0402_1005_DensityHigh, F.Cu at (26.9, 42.2)
- added C2102: 1n X7R 1kV, 0_capacitor_smd:C_0603_1608_DensityHigh, F.Cu at (248.7, 84.2)
- added C2103: 1n X7R 1kV, 0_capacitor_smd:C_0603_1608_DensityHigh, F.Cu at (50.4, 106.5)
- added C2104: 1n X7R 1kV, 0_capacitor_smd:C_0603_1608_DensityHigh, F.Cu at (248.7, 106.5)
- added C2105: 1n X7R 1kV, 0_capacitor_smd:C_0603_1608_DensityHigh, F.Cu at (51.8, 84.2)
- added C2201: 1n X7R 1kV, 0_capacitor_smd:C_0603_1608_DensityHigh, F.Cu at (51.2, 61.3)
- added C2202: 1n X7R 1kV, 0_capacitor_smd:C_0603_1608_DensityHigh, F.Cu at (51.1, 115.8)
- added C2203: 1n X7R 1kV, 0_capacitor_smd:C_0603_1608_DensityHigh, F.Cu at (249.5, 115.8)
- added C2204: 1n X7R 1kV, 0_capacitor_smd:C_0603_1608_DensityHigh, F.Cu at (249.4, 61.2)
- added C2501: 100n X7R 50V, 0_capacitor_smd:C_0402_1005_DensityHigh, F.Cu at (116.2, 97.4)
- added C2503: 100n X7R 50V, 0_capacitor_smd:C_0402_1005_DensityHigh, F.Cu at (126.0, 97.4)
- added C2505: 100n X7R 50V, 0_capacitor_smd:C_0402_1005_DensityHigh, F.Cu at (116.2, 95.8)
- added C401: 12p NP0 25V, Capacitor_SMD:C_0402_1005Metric, F.Cu at (147.4, 101.9)
- added C402: 12p NP0 25V, Capacitor_SMD:C_0402_1005Metric, F.Cu at (146.1, 103.3)
- added C403: 100n X7R 50V, 0_capacitor_smd:C_0402_1005_DensityHigh, F.Cu at (204.3, -22.0)
- added C404: 100n X7R 50V, 0_capacitor_smd:C_0402_1005_DensityHigh, F.Cu at (187.4, 59.6)
- added C405: 100n X7R 50V, 0_capacitor_smd:C_0402_1005_DensityHigh, F.Cu at (192.4, 59.8)
- added C406: 1u X7R 10V, 0_capacitor_smd:C_0402_1005_DensityHigh, F.Cu at (148.5, 117.1)
- added C407: 100n X7R 50V, 0_capacitor_smd:C_0402_1005_DensityHigh, F.Cu at (158.6, 111.2)
- added C408: 100n X7R 50V, 0_capacitor_smd:C_0402_1005_DensityHigh, F.Cu at (143.2, 106.3)
- added C409: 100n X7R 50V, 0_capacitor_smd:C_0402_1005_DensityHigh, F.Cu at (148.8, 100.8)
- added C410: 100n X7R 50V, 0_capacitor_smd:C_0402_1005_DensityHigh, F.Cu at (153.5, 101.3)
- added C411: 4u7 X7R 16V, 0_capacitor_smd:C_0603_1608_DensityHigh, F.Cu at (154.6, 100.8)
- added C412: 1u X7R 10V, 0_capacitor_smd:C_0402_1005_DensityHigh, F.Cu at (143.7, 114.8)
- added C413: 1u X7R 10V, 0_capacitor_smd:C_0402_1005_DensityHigh, F.Cu at (146.0, 115.3)
- added C414: 100n X7R 50V, 0_capacitor_smd:C_0402_1005_DensityHigh, F.Cu at (146.6, 114.7)
- added C415: 1u X7R 10V, 0_capacitor_smd:C_0402_1005_DensityHigh, F.Cu at (147.2, 116.4)
- added C416: 100n X7R 50V, 0_capacitor_smd:C_0402_1005_DensityHigh, F.Cu at (147.7, 115.8)
- added C801: 2u2 X7R 100V, 0_capacitor_smd:C_0805_2012_DensityHigh, F.Cu at (127.3, 145.7)
- added C802: 100n X7R 100V, 0_capacitor_smd:C_0805_2012_DensityHigh, F.Cu at (129.1, 145.7)
- added C803: 10u X7R 25V, 0_capacitor_smd:C_1210_3225_DensityHigh, F.Cu at (137.7, 141.4)
- added C804: 2.2u X7R 25V, 0_capacitor_smd:C_0805_2012_DensityHigh, F.Cu at (126.2, 140.9)
- added C805: 2.2u X7R 25V, 0_capacitor_smd:C_0805_2012_DensityHigh, F.Cu at (140.1, 140.9)
- added D1101: PESD4USB5B-TBSX, 0_package_DFN_QFN:SOT1176D, B.Cu at (94.2, 60.1)
- added D1102: PESD2CANFD24V-UX, 0_package_SOT_TO_SMD:SOT95P230X117-3N, F.Cu at (179.9, 67.8)
- added D1103: PESD2CANFD24V-UX, 0_package_SOT_TO_SMD:SOT95P230X117-3N, F.Cu at (177.3, 67.8)
- added D1104: PESD2CANFD24V-UX, 0_package_SOT_TO_SMD:SOT95P230X117-3N, F.Cu at (120.3, 67.7)
- added D1105: PESD2CANFD24V-UX, 0_package_SOT_TO_SMD:SOT95P230X117-3N, F.Cu at (122.9, 67.7)
- added D1106: PESD4USB5B-TBSX, 0_package_DFN_QFN:SOT1176D, B.Cu at (68.1, 60.2)
- added D1107: ORANGE, 0_led_smd:LED_SM1206, F.Cu at (164.5, 88.3)
- added D1301: PESD4USB5B-TBSX, 0_package_DFN_QFN:SOT1176D, F.Cu at (178.0, 95.6)
- added D1302: PESD4USB5B-TBSX, 0_package_DFN_QFN:SOT1176D, F.Cu at (178.0, 98.5)
- added D1401: PESD4USB5B-TBSX, 0_package_DFN_QFN:SOT1176D, F.Cu at (126.5, 92.3)
- added D1501: SMBJ51CD-M3/H, 0_diode_smd:DIOM4336X24N, F.Cu at (110.0, -52.3)
- added D1503: SMBJ51CD-M3/H, 0_diode_smd:DIOM4336X24N, F.Cu at (110.0, -47.4)
- added D1901: YELLOW, LED_SMD:LED_0603_1608Metric, F.Cu at (178.4, -20.7)
- added D1902: GREEN, LED_SMD:LED_0603_1608Metric, F.Cu at (178.4, -18.1)
- added D1903: USB, LED_SMD:LED_0603_1608Metric, F.Cu at (178.4, -15.5)
- added D2501: PESD4USB5B-TBSX, 0_package_DFN_QFN:SOT1176D, F.Cu at (126.5, 95.1)
- added D401: PRTR5V0U2X, Package_TO_SOT_SMD:SOT-143, F.Cu at (109.8, 63.5)
- added D402: PESD4USB3U-TBSX, 0_package_DFN_QFN:SOT1176D, F.Cu at (190.5, 59.8)
- added D501: SMBJ51CD-M3/H, 0_diode_smd:DIOM4336X24N, F.Cu at (107.5, 71.8)
- added D502: SMBJ51CD-M3/H, 0_diode_smd:DIOM4336X24N, F.Cu at (107.5, 75.8)
- added D503: SMBJ51CD-M3/H, 0_diode_smd:DIOM4336X24N, F.Cu at (23.8, 32.3)
- added D504: SMBJ51CD-M3/H, 0_diode_smd:DIOM4336X24N, F.Cu at (27.8, 32.3)
- added F1301: 0451015.MRL, 0_diode_smd:FUSC6127X294N, F.Cu at (189.7, 99.7)
- added F1401: 0451015.MRL, 0_diode_smd:FUSC6127X294N, F.Cu at (114.8, 91.1)
- added FB1101: BLM18PG330SN1D, 0_diode_smd:BLM18SP221SN1B, F.Cu at (150.3, 81.2)
- added FB1102: BLM18PG330SN1D, 0_diode_smd:BLM18SP221SN1B, F.Cu at (155.7, 85.1)
- added FB1103: BLM18PG330SN1D, 0_diode_smd:BLM18SP221SN1B, F.Cu at (144.9, 85.1)
- added FB1104: BLM18PG330SN1D, 0_diode_smd:BLM18SP221SN1B, F.Cu at (157.4, 95.8)
- added FB1201: 1k @ 100MHz, 0_resistor_smd:R_0805_2012_DensityHigh, F.Cu at (174.5, 135.4)
- added FB401: 100R@100MHz, Inductor_SMD:L_0603_1608Metric, F.Cu at (145.2, 116.1)
- added FM2201: Fiducial, 0_fiducials:Fiducial_1mm_Mask2mm, B.Cu at (125.3, 121.9)
- added FM2202: Fiducial, 0_fiducials:Fiducial_1mm_Mask2mm, F.Cu at (125.3, 121.9)
- added FM2203: Fiducial, 0_fiducials:Fiducial_1mm_Mask2mm, B.Cu at (175.3, 121.9)
- added FM2204: Fiducial, 0_fiducials:Fiducial_1mm_Mask2mm, F.Cu at (150.3, 63.7)
- added FM2205: Fiducial, 0_fiducials:Fiducial_1mm_Mask2mm, B.Cu at (150.3, 63.7)
- added FM2206: Fiducial, 0_fiducials:Fiducial_1mm_Mask2mm, F.Cu at (175.3, 121.9)
- added H2101: M2 (3.2mm), MountingHole:MountingHole_2.2mm_M2_Pad_Via, F.Cu at (249.4, 80.4)
- added H2102: M2 (3.2mm), MountingHole:MountingHole_2.2mm_M2_Pad_Via, F.Cu at (249.4, 110.4)
- added H2103: M2 (3.2mm), MountingHole:MountingHole_2.2mm_M2_Pad_Via, F.Cu at (51.1, 80.4)
- added H2104: M2 (3.2mm), MountingHole:MountingHole_2.2mm_M2_Pad_Via, F.Cu at (51.1, 110.4)
- added H2201: M3 (3.2mm), MountingHole:MountingHole_3.2mm_M3_Pad_Via, F.Cu at (51.8, 56.4)
- added H2202: M3 (3.2mm), MountingHole:MountingHole_3.2mm_M3_Pad_Via, F.Cu at (51.8, 120.5)
- added H2203: M3 (3.2mm), MountingHole:MountingHole_3.2mm_M3_Pad_Via, F.Cu at (248.8, 120.6)
- added H2204: M3 (3.2mm), MountingHole:MountingHole_3.2mm_M3_Pad_Via, F.Cu at (248.8, 56.4)
- added IC1101: LAN9252_ML, 0_package_SOT_TO_SMD:QFN50P900X900X100-65N-D, F.Cu at (150.8, 92.0)
- added IC1102: M24C16-RMN6P, 0_package_SOT_TO_SMD:SOIC127P600X175-8N, F.Cu at (163.0, 92.3)
- added IC1201: MAX25262AFOF_VY+, 0_switching_regulator:MAX25262AFOFVY, F.Cu at (133.1, 147.5)
- added IC1202: TPS629206QDRLRQ1, 0_switching_regulator:SOTFL50P160X60-8N, F.Cu at (130.0, 134.7)
- added IC1203: TPS7A2650DRVR, 0_switching_regulator:SON65P200X200X80-7N, F.Cu at (134.4, 134.6)
- added IC1501: TPS2490DGSRG4, 0_connectors:SOP50P490X110-10N, F.Cu at (25.1, 44.5)
- added IC1701: TPA6205A1DGN, 0_connectors:SOP65P490X110-9N, F.Cu at (206.3, -12.5)
- added IC2001: INA239AQDGSRQ1, 0_diode_smd:SOP50P490X110-10N, F.Cu at (25.1, 40.0)
- added J1101: SM07B-GHS-TB, 0_connectors:JST_GH_SM07B-GHS-TB_1x07-1MP_P1.25mm_Horizontal, B.Cu at (93.6, 55.9)
- added J1102: Nano-Fit 1x03, 0_connectors:1054301203, B.Cu at (121.6, 58.9)
- added J1103: Nano-Fit 1x03, 0_connectors:1054301203, F.Cu at (121.6, 58.9)
- added J1104: Nano-Fit 1x03, 0_connectors:1054301203, F.Cu at (178.6, 58.9)
- added J1105: Nano-Fit 1x03, 0_connectors:1054301203, B.Cu at (178.6, 58.9)
- added J1106: SM07B-GHS-TB, 0_connectors:JST_GH_SM07B-GHS-TB_1x07-1MP_P1.25mm_Horizontal, B.Cu at (67.5, 55.9)
- added J1107: RJ45_Wuerth_74980111211, Connector_RJ:RJ45_Wuerth_74980111211_Horizontal, F.Cu at (161.3, 65.9)
- added J1108: RJ45_Wuerth_74980111211, Connector_RJ:RJ45_Wuerth_74980111211_Horizontal, F.Cu at (139.2, 65.9)
- added J1109: PTH 01x03 2.54mm, 0_connectors:PTH_1x03_P2.54mm, F.Cu at (121.7, 35.2)
- added J1110: PTH 01x03 2.54mm, 0_connectors:PTH_1x03_P2.54mm, F.Cu at (184.8, 35.1)
- added J1301: 10159558-410421RLF, 0_connectors:10159558410421RLF, F.Cu at (183.4, 95.4)
- added J1701: 53048-0450, 0_connectors:SHDRRA4W35P0X125_1X4_675X550X350P, F.Cu at (135.7, -44.6)
- added J1702: 505110-3091, 0_connectors:5051103091, F.Cu at (137.8, -33.0)
- added J1801: Screw_Terminal_01x02, 0_connectors:JST_PH_S2B-PH-SM4-TB_1x02-1MP_P2.00mm_Horizontal, F.Cu at (165.1, -19.0)
- added J2501: 10159558-410421RLF, 0_connectors:10159558410421RLF, F.Cu at (121.1, 95.4)
- added J301: Rail 1, 0_pad:Pad_Square_Vias_6.5x6.5mm, F.Cu at (239.3, 80.5)
- added J302: Rail 2, 0_pad:Pad_Square_Vias_6.5x6.5mm, F.Cu at (227.1, 80.5)
- added J303: Rail 3, 0_pad:Pad_Square_Vias_6.5x6.5mm, F.Cu at (215.0, 80.5)
- added J304: Rail 4, 0_pad:Pad_Square_Vias_6.5x6.5mm, F.Cu at (202.7, 80.5)
- added J305: Vin, 0_pad:Pad_Square_Vias_6.5x6.5mm, F.Cu at (105.6, 146.4)
- added J402: Conn_Picoblade_JST_DEBUG, 0_connectors:CONN_SM06B-GHS-TB_JST, F.Cu at (190.5, 55.8)
- added J403: USB4105-GF-A, Connector_USB:USB_C_Receptacle_GCT_USB4105-xx-A_16P_TopMnt_Horizontal, F.Cu at (110.0, 56.9)
- added J501: XT90PW-M, 0_connectors:XT90pw-m, F.Cu at (93.8, 65.3)
- added J502: XT90PW-F, 0_connectors:XT90PW-F, F.Cu at (67.6, 65.3)
- added L1202: 2.2uH, 0_switching_regulator:IND_XGL3530_COC, F.Cu at (130.0, 131.4)
- added L801: 3.3uH, 0_switching_regulator:XEL4030682MEC, F.Cu at (133.1, 141.2)
- added Molex_601: ~, 0_connectors:172448-YY02, F.Cu at (241.8, 67.0)
- added Molex_602: ~, 0_connectors:172448-YY02, F.Cu at (235.8, 67.0)
- added Molex_603: ~, 0_connectors:172448-YY02, F.Cu at (229.8, 67.0)
- added Molex_604: ~, 0_connectors:172448-YY02, F.Cu at (223.8, 67.0)
- added Molex_605: ~, 0_connectors:172448-YY02, F.Cu at (217.8, 67.0)
- added Molex_606: ~, 0_connectors:172448-YY02, F.Cu at (211.8, 67.0)
- added Molex_607: ~, 0_connectors:172448-YY02, F.Cu at (205.8, 67.0)
- added Molex_608: ~, 0_connectors:172448-YY02, F.Cu at (199.7, 67.0)
- added NT1101: NetTieShuntH, 0_net_tie:NetTie-2_SMD_Pad0.2mm, F.Cu at (91.2, 80.2)
- added NT1103: NetTieShuntL, 0_net_tie:NetTie-2_SMD_Pad0.2mm, F.Cu at (89.6, 80.2)
- added NT1601: NetTieShuntH, 0_net_tie:NetTie-2_SMD_Pad0.2mm, F.Cu at (91.2, 81.0)
- added NT1602: NetTieShuntL, 0_net_tie:NetTie-2_SMD_Pad0.2mm, F.Cu at (89.6, 81.0)
- added Q1601: PSMN4R8-100BSEJ, 0_diode_smd:PHB45NQ15T118, F.Cu at (88.2, 117.4)
- added Q1602: PSMN4R8-100BSEJ, 0_diode_smd:PHB45NQ15T118, F.Cu at (88.2, 104.6)
- added Q1603: PSMN4R8-100BSEJ, 0_diode_smd:PHB45NQ15T118, F.Cu at (88.2, 91.8)
- added Q1604: PSMN4R8-100BSEJ, 0_diode_smd:PHB45NQ15T118, F.Cu at (72.7, 117.4)
- added Q1605: PSMN4R8-100BSEJ, 0_diode_smd:PHB45NQ15T118, F.Cu at (72.7, 104.6)
- added Q1606: PSMN4R8-100BSEJ, 0_diode_smd:PHB45NQ15T118, F.Cu at (72.7, 91.8)
- added Q1801: PMV90ENER, 0_package_SOT_TO_SMD:SOT-23-3, F.Cu at (193.8, -16.7)
- added R1101: 10k 1% 1/16W, 0_resistor_smd:R_0402_1005_DensityHigh, F.Cu at (129.1, 48.1)
- added R1102: 10k 1% 1/16W, 0_resistor_smd:R_0402_1005_DensityHigh, F.Cu at (177.4, 44.1)
- added R1103: 100R 1% 1/5W, 0_resistor_smd:R_0402_1005_DensityHigh, B.Cu at (92.2, 62.1)
- added R1104: 100R 1% 1/5W, 0_resistor_smd:R_0402_1005_DensityHigh, B.Cu at (93.0, 62.1)
- added R1105: 100R 1% 1/5W, 0_resistor_smd:R_0402_1005_DensityHigh, B.Cu at (95.5, 62.1)
- added R1106: 100R 1% 1/5W, 0_resistor_smd:R_0402_1005_DensityHigh, B.Cu at (96.3, 62.1)
- added R1107: 60R4 1% 1/4W, 0_resistor_smd:R_0603_1608_DensityHigh, F.Cu at (179.4, 38.7)
- added R1108: 60R4 1% 1/4W, 0_resistor_smd:R_0603_1608_DensityHigh, F.Cu at (182.5, 38.7)
- added R1109: 100R 1% 1/5W, 0_resistor_smd:R_0402_1005_DensityHigh, B.Cu at (66.0, 62.2)
- added R1110: 100R 1% 1/5W, 0_resistor_smd:R_0402_1005_DensityHigh, B.Cu at (66.9, 62.2)
- added R1111: 100R 1% 1/5W, 0_resistor_smd:R_0402_1005_DensityHigh, B.Cu at (69.3, 62.2)
- added R1112: 100R 1% 1/5W, 0_resistor_smd:R_0402_1005_DensityHigh, B.Cu at (70.2, 62.2)
- added R1113: 4.75k 0.1% 1/16W, 0_resistor_smd:R_0402_1005_DensityHigh, F.Cu at (142.3, 93.6)
- added R1114: 4.75k 0.1% 1/16W, 0_resistor_smd:R_0402_1005_DensityHigh, F.Cu at (150.4, 76.4)
- added R1115: 4.75k 0.1% 1/16W, 0_resistor_smd:R_0402_1005_DensityHigh, F.Cu at (144.1, 92.7)
- added R1116: 12k 1%, 1/16W, 0_resistor_smd:R_0402_1005_DensityHigh, F.Cu at (150.7, 84.5)
- added R1117: 49.9R 0.1% 1/16W, 0_resistor_smd:R_0402_1005_DensityHigh, F.Cu at (157.8, 82.5)
- added R1118: 49.9R 0.1% 1/16W, 0_resistor_smd:R_0402_1005_DensityHigh, F.Cu at (135.8, 84.8)
- added R1119: 49.9R 0.1% 1/16W, 0_resistor_smd:R_0402_1005_DensityHigh, F.Cu at (159.6, 82.5)
- added R1120: 49.9R 0.1% 1/16W, 0_resistor_smd:R_0402_1005_DensityHigh, F.Cu at (137.5, 84.8)
- added R1121: 49.9R 0.1% 1/16W, 0_resistor_smd:R_0402_1005_DensityHigh, F.Cu at (160.9, 84.9)
- added R1122: 49.9R 0.1% 1/16W, 0_resistor_smd:R_0402_1005_DensityHigh, F.Cu at (138.8, 82.5)
- added R1123: 49.9R 0.1% 1/16W, 0_resistor_smd:R_0402_1005_DensityHigh, F.Cu at (162.7, 84.9)
- added R1124: 49.9R 0.1% 1/16W, 0_resistor_smd:R_0402_1005_DensityHigh, F.Cu at (140.6, 82.5)
- added R1125: 470R 1% 1/16W, 0_resistor_smd:R_0402_1005_DensityHigh, F.Cu at (161.6, 88.3)
- added R1126: 10R 1% 1/8W, 0_resistor_smd:R_0603_1608_DensityHigh, F.Cu at (165.6, 83.3)
- added R1127: 10R 1% 1/8W, 0_resistor_smd:R_0603_1608_DensityHigh, F.Cu at (132.9, 83.3)
- added R1128: 4.75k 0.1% 1/16W, 0_resistor_smd:R_0402_1005_DensityHigh, F.Cu at (157.4, 90.2)
- added R1129: 4.75k 0.1% 1/16W, 0_resistor_smd:R_0402_1005_DensityHigh, F.Cu at (157.4, 91.8)
- added R1130: 4.75k 0.1% 1/16W, 0_resistor_smd:R_0402_1005_DensityHigh, F.Cu at (158.8, 93.2)
- added R1131: 470R 1% 1/16W, 0_resistor_smd:R_0402_1005_DensityHigh, F.Cu at (167.9, 82.9)
- added R1132: 470R 1% 1/16W, 0_resistor_smd:R_0402_1005_DensityHigh, F.Cu at (152.2, 81.2)
- added R1133: 470R 1% 1/16W, 0_resistor_smd:R_0402_1005_DensityHigh, F.Cu at (148.3, 81.2)
- added R1134: 470R 1% 1/16W, 0_resistor_smd:R_0402_1005_DensityHigh, F.Cu at (131.2, 83.0)
- added R1135: 4.75k 0.1% 1/16W, 0_resistor_smd:R_0402_1005_DensityHigh, F.Cu at (152.7, 82.6)
- added R1136: 4.75k 0.1% 1/16W, 0_resistor_smd:R_0402_1005_DensityHigh, F.Cu at (131.6, 87.1)
- added R1138: 60R4 1% 1/4W, 0_resistor_smd:R_0603_1608_DensityHigh, F.Cu at (124.0, 38.3)
- added R1139: 60R4 1% 1/4W, 0_resistor_smd:R_0603_1608_DensityHigh, F.Cu at (127.1, 38.3)
- added R1201: 10k 1% 1/16W, 0_resistor_smd:R_0402_1005_DensityHigh, F.Cu at (136.6, 148.9)
- added R1202: 34k 1% 1/4W, 0_resistor_smd:R_0603_1608_DensityHigh, F.Cu at (131.6, 136.9)
- added R1501: 212k 1% 1/10W, 0_resistor_smd:R_0603_1608_DensityHigh, F.Cu at (26.8, 63.4)
- added R1502: 10k 1% 1/4W, 0_resistor_smd:R_1206_3216_DensityHigh_Large, F.Cu at (17.9, 43.5)
- added R1503: 45k 1% 1/10W, 0_resistor_smd:R_0603_1608_DensityHigh, F.Cu at (20.5, 44.5)
- added R1504: 7,5k 1% 1/4W, 0_resistor_smd:R_1206_3216_DensityHigh_Large, F.Cu at (17.9, 45.5)
- added R1505: 0.3m, 0_resistor_smd:RES_WSLP3921_.003OHM_VIS, F.Cu at (90.4, 80.6)
- added R1507: 1k 1% 1/10W, 0_resistor_smd:R_0603_1608_DensityHigh, F.Cu at (-37.8, 94.8)
- added R1601: 10R 1% 1/8W, 0_resistor_smd:R_0805_2012_DensityHigh, F.Cu at (-37.8, 127.0)
- added R1602: 10R 1% 1/8W, 0_resistor_smd:R_0805_2012_DensityHigh, F.Cu at (-37.8, 114.2)
- added R1603: 10R 1% 1/8W, 0_resistor_smd:R_0805_2012_DensityHigh, F.Cu at (-37.8, 101.3)
- added R1604: 10R 1% 1/8W, 0_resistor_smd:R_0805_2012_DensityHigh, F.Cu at (-37.8, 121.8)
- added R1605: 10R 1% 1/8W, 0_resistor_smd:R_0805_2012_DensityHigh, F.Cu at (-37.8, 109.0)
- added R1606: 10R 1% 1/8W, 0_resistor_smd:R_0805_2012_DensityHigh, F.Cu at (-37.8, 96.3)
- added R1701: 33 1% 1/10W, 0_resistor_smd:R_0603_1608_DensityHigh, F.Cu at (210.7, -24.8)
- added R1702: 33 1% 1/10W, 0_resistor_smd:R_0603_1608_DensityHigh, F.Cu at (108.7, -29.1)
- added R1703: 1k 1% 1/10W, 0_resistor_smd:R_0603_1608_DensityHigh, F.Cu at (209.8, -18.0)
- added R1704: 1k 1% 1/10W, 0_resistor_smd:R_0603_1608_DensityHigh, F.Cu at (209.8, -15.6)
- added R1705: 47k 1% 1/10W, 0_resistor_smd:R_0603_1608_DensityHigh, F.Cu at (108.7, -22.6)
- added R1706: 1k 1% 1/10W, 0_resistor_smd:R_0603_1608_DensityHigh, F.Cu at (209.8, -13.1)
- added R1707: 10k 1% 1/10W, 0_resistor_smd:R_0603_1608_DensityHigh, F.Cu at (203.8, -10.7)
- added R1708: 10k 1% 1/10W, 0_resistor_smd:R_0603_1608_DensityHigh, F.Cu at (209.3, -9.92)
- added R1709: 20k 1% 1/10W, 0_resistor_smd:R_0603_1608_DensityHigh, F.Cu at (209.3, -11.2)
- added R1710: 20k 1% 1/10W, 0_resistor_smd:R_0603_1608_DensityHigh, F.Cu at (203.8, -13.1)
- added R1901: 768R 1% 1/8W, Resistor_SMD:R_0603_1608Metric, F.Cu at (182.4, -20.7)
- added R1902: 40R 5% 1/4W, Resistor_SMD:R_0603_1608Metric, F.Cu at (182.4, -18.2)
- added R1903: 40R 5% 1/4W, Resistor_SMD:R_0603_1608Metric, F.Cu at (182.4, -15.7)
- added R2102: 0R, 0_resistor_smd:R_0603_1608_DensityHigh, F.Cu at (250.0, 84.2)
- added R2103: 0R, 0_resistor_smd:R_0603_1608_DensityHigh, F.Cu at (51.7, 106.5)
- added R2104: 0R, 0_resistor_smd:R_0603_1608_DensityHigh, F.Cu at (250.0, 106.5)
- added R2105: 0R, 0_resistor_smd:R_0603_1608_DensityHigh, F.Cu at (50.5, 84.2)
- added R2201: 0R, 0_resistor_smd:R_0603_1608_DensityHigh, F.Cu at (52.5, 61.3)
- added R2202: 0R, 0_resistor_smd:R_0603_1608_DensityHigh, F.Cu at (52.4, 115.8)
- added R2203: 0R, 0_resistor_smd:R_0603_1608_DensityHigh, F.Cu at (248.2, 115.8)
- added R2204: 0R, 0_resistor_smd:R_0603_1608_DensityHigh, F.Cu at (248.2, 61.2)
- added R401: 33k 1% 1/16W, 0_resistor_smd:R_0402_1005_DensityHigh, F.Cu at (144.9, 113.7)
- added R402: 5.1k 1% 1/16W, 0_resistor_smd:R_0402_1005_DensityHigh, F.Cu at (111.9, 62.5)
- added R403: 5.1k 1% 1/16W, 0_resistor_smd:R_0402_1005_DensityHigh, F.Cu at (107.7, 62.5)
- added R404: 10k 1% 1/16W, 0_resistor_smd:R_0402_1005_DensityHigh, F.Cu at (157.4, 104.7)
- added R405: 10k 1% 1/16W, 0_resistor_smd:R_0402_1005_DensityHigh, F.Cu at (143.8, 112.6)
- added R406: 10k 1% 1/16W, 0_resistor_smd:R_0402_1005_DensityHigh, F.Cu at (154.6, 115.8)
- added R407: 27R 1% 1/5W, 0_resistor_smd:R_0402_1005_DensityHigh, F.Cu at (110.2, 66.0)
- added R408: 27R 1% 1/5W, 0_resistor_smd:R_0402_1005_DensityHigh, F.Cu at (109.4, 66.0)
- added SW1101: CAS-220TA, 0_switch_button:CAS-220A_NDC-L, F.Cu at (181.0, 42.2)
- added SW1103: CAS-220TA, 0_switch_button:CAS-220A_NDC-L, F.Cu at (125.5, 41.8)
- added U1101: TCAN1051HGVDRBRQ1, 0_package_SON:HVSON-8-1EP_3x3mm_P0.65mm_EP1.6x2.4mm_ThermalVias, F.Cu at (129.9, 45.9)
- added U1102: TCAN1051HGVDRBRQ1, 0_package_SON:HVSON-8-1EP_3x3mm_P0.65mm_EP1.6x2.4mm_ThermalVias, F.Cu at (176.7, 46.3)
- added U1701: 74LVC1G125, 0_package_SON:SOT95P280X145-5N, F.Cu at (210.7, -21.4)
- added U1801: DGD0216WT-7, Package_TO_SOT_SMD:TSOT-23-5, F.Cu at (139.8, -10.7)
- added U401: STM32G483RET6, Package_QFP:LQFP-64_10x10mm_P0.5mm, F.Cu at (150.8, 108.8)
- added Y1101: 7M-25.000MAAJ-T, 0_switch_button:7M25000MAAJT, F.Cu at (140.6, 89.5)
- added Y401: ABM8W-48.0000MHZ-4-D1X-T3, 0_diode_smd:ABM8W480000MHZ6D1XT3, F.Cu at (144.5, 100.3)
Routing:
- net /Project Architecture/Connectors - Communication/FDCAN1_N: track 0.00 -> 42.3 mm, vias 0 -> 2
- net /Project Architecture/Connectors - Communication/FDCAN1_P: track 0.00 -> 40.1 mm, vias 0 -> 2
- net /Project Architecture/Connectors - Communication/FDCAN2_N: track 0.00 -> 39.2 mm, vias 0 -> 2
- net +3V3: track 0.00 -> 38.6 mm, vias 0 -> 22
- net /Project Architecture/Connectors - Communication/FDCAN2_P: track 0.00 -> 38.4 mm, vias 0 -> 2
- net Net-(Q1601-G): track 0.00 -> 37.4 mm, vias 0 -> 2
- net Net-(Q1603-G): track 0.00 -> 37.3 mm, vias 0 -> 2
- net Net-(Q1602-G): track 0.00 -> 37.3 mm, vias 0 -> 2
- net /Project Architecture/Connectors - Communication/LED_ON2: track 0.00 -> 35.3 mm, vias 0 -> 2
- net /Project Architecture/Power - Precharge/Power - MOS/G: track 0.00 -> 32.8 mm, vias 0 -> 1
- net Net-(C1111-Pad1): track 0.00 -> 30.9 mm, vias 0 -> 4
- net /Project Architecture/Connectors - Communication/RXA_N: track 0.00 -> 25.7 mm, vias 0 -> 2
- net /Project Architecture/Connectors - Communication/RXA_P: track 0.00 -> 25.7 mm, vias 0 -> 2
- net /Project Architecture/Connectors - Communication/TXB_P: track 0.00 -> 25.2 mm, vias 0 -> 2
- net Net-(IC1101-VDD12TX1): track 0.00 -> 24.7 mm, vias 0 -> 3
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- added copper zone on F.Cu, net +12V
- added copper zone on F.Cu, net +3.3VA
- added copper zone on F.Cu, net +3V3
- added copper zone on In2.Cu, net +3V3
- added copper zone on In2.Cu, net +3V3_A
- added copper zone on In2.Cu, net +3V3_B
- added copper zone on F.Cu, net +5V
- added copper zone on B.Cu, net +VBAT
- added copper zone on F.Cu, net +VBAT
- added copper zone on In2.Cu, net +VBAT
- added copper zone on In3.Cu, net +VBAT
- added copper zone on B.Cu, net +VIN
- added copper zone on F.Cu, net +VIN
- added copper zone on In2.Cu, net +VIN
- added copper zone on In3.Cu, net +VIN
- added copper zone on F.Cu, net /Project Architecture/Connectors - Communication/FDCAN1_S
- added copper zone on F.Cu, net /Project Architecture/Power - Precharge/Vsense_low
- added copper zone on B.Cu, net GND
- added copper zone on F.Cu, net GND
- added copper zone on In1.Cu, net GND
- added copper zone on In4.Cu, net GND
- added copper zone on F.Cu, net Net-(C2102-Pad1)
- added copper zone on F.Cu, net Net-(C2103-Pad1)
- added copper zone on F.Cu, net Net-(C2104-Pad1)
- added copper zone on F.Cu, net Net-(C2105-Pad1)
- added copper zone on F.Cu, net Net-(C2201-Pad1)
- added copper zone on F.Cu, net Net-(C2202-Pad1)
- added copper zone on F.Cu, net Net-(C2203-Pad1)
- added copper zone on F.Cu, net Net-(C2204-Pad1)
- added copper zone on F.Cu, net Net-(IC1201-BIAS)
- added copper zone on F.Cu, net Net-(IC1201-EN)
- added copper zone on F.Cu, net Net-(IC1201-LX)
- added copper zone on F.Cu, net Net-(IC1202-SW)
Other:
- board outline added: 204.5 x 71.7 mm

Commit message: Correction module
Parts:
- added REF**: Module_step, 0_pad:Module_step, F.Cu at (250.9, 77.2)
- added REF**: Module_step, 0_pad:Module_step, F.Cu at (49.6, 113.3)
- J501: footprint 0_connectors:XT90pw-m -> 0_connectors:AMASS_XT90PW-M
- J502: footprint 0_connectors:XT90PW-F -> 0_connectors:AMASS_XT90PW-F
- moved C1301 6.00 mm to (182.3, 93.4)
- moved C1302 6.00 mm to (183.7, 104.2)
- moved C1303 6.00 mm to (172.5, 93.4)
- moved C1305 6.00 mm to (182.3, 95.0)
- moved D1301 6.00 mm to (172.0, 95.6)
- moved D1302 6.00 mm to (172.0, 98.5)
- moved F1301 6.00 mm to (183.7, 99.7)
- moved J1301 6.00 mm to (177.4, 95.4)
- moved C1401 2.00 mm to (116.8, 86.6)
- moved C2501 2.00 mm to (118.2, 97.4)
- moved C2503 2.00 mm to (128.0, 97.4)
- moved C2505 2.00 mm to (118.2, 95.8)
- moved D2501 2.00 mm to (128.5, 95.1)
- moved F1401 2.00 mm to (116.8, 91.1)
- moved J2501 2.00 mm to (123.1, 95.4)
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Connections:
- J502 pad 1: GND -> (no net)
- J502 pad 2: +VIN -> (no net)
- NT1601 pad 2: +VBAT -> /Project Architecture/Power - Precharge/VBAT_IN
