File: amulet_controller/Schematic/value_split/Interface - Interconnects.kicad_sch (KiCad schematic)
At the start: 57 parts, among them J10 SM06B-GHS-TB, J11 PTH 01x03 2.54mm, J12 Nano-Fit 1x03, J13 Nano-Fit 1x03, J14 SM05B-GHS-TB, J6 SM08B-GHS-TB, J7 SM07B-GHS-TB, J8 S2B-PH-SM4-TB, J9 S2B-PH-SM4-TB, SW1 CAS-220TA

Commit message: Better syntax for fab copper layers and testpoints
Parts:
- J7: manf# SM07B-GHS-TB -> SM07B-GHS-TB(LF)(SN)
Changed lines of the file:
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@@
       (effects (font (size 1.27 1.27)) (hide yes))
     )
-    (property "manf#" "SM07B-GHS-TB" (at 50.8 176.53 0)
+    (property "manf#" "SM07B-GHS-TB(LF)(SN)" (at 50.8 176.53 0)
       (effects (font (size 1.27 1.27)) (hide yes))
     )
